Commit message: F3D, Force and Odometry Plugins added

File: grips_description/robots/grips_robotiq.xacro (robot description, xacro)
@@ -12,5 +12,5 @@
   <xacro:include filename="$(find grips_description)/urdf/imu_sensor.xacro" />
   <!-- Import robotiq s model -->
-  <xacro:include filename="$(find robotiq_s_model_visualization)/cfg/s-model_fixed_macro.xacro" />
+  <xacro:include filename="$(find robotiq_s_model_visualization)/cfg/s-model_articulated.xacro" />
   <property name="robot_name" value="" />
   <!-- Create the grips robot -->
@@ -20,5 +20,5 @@
   <!-- Add the imu_sensor -->
   <imu_sensor prefix="${robot_name}" parent="${robot_name}end_effector">
-    <origin xyz="0 0.13 ${board_z_size+63.635e-3}" rpy="0 0 ${-pi/2}" />
+    <origin xyz="0 0.13 ${board_z_size+63.635e-3}" rpy="0 0 0" />
   </imu_sensor>
   <!-- Add robotiq hand -->
@@ -47,3 +47,33 @@
     </plugin>
   </gazebo>
+  <!--ROS P3D odometry -->
+	<gazebo>
+		<plugin name="imu_sensor_odometry" filename="libgazebo_ros_p3d.so">
+			<robotNamespace>/grips</robotNamespace>
+			<bodyName>end_effector</bodyName>
+			<topicName>imu_odom</topicName>
+			<frameName>base_link</frameName>
+			<xyzOffset>0 0 0</xyzOffset>
+			<rpyOffset>0 0 0</rpyOffset>
+			<gaussianNoise>0.0</gaussianNoise>
+			<updateRate>1000</updateRate>
+		</plugin>
+	</gazebo>
+	<!-- ROS Force Plugin -->
+	<gazebo>
+		<plugin name="ext_force_publisher" filename="libgazebo_ros_force.so">
+			<robotNamespace>/grips</robotNamespace>
+			<bodyName>end_effector</bodyName>
+			<topicName>ext_force</topicName>
+		</plugin>
+	</gazebo>
+	<!-- ROS F3D Plugin -->
+	<gazebo>
+		<plugin name="ext_force_listener" filename="libgazebo_ros_f3d.so">
+			<robotNamespace>/grips</robotNamespace>
+			<topicName>extft_data</topicName>
+			<bodyName>end_effector</bodyName>
+			<frameName>base_link</frameName>
+		</plugin>
+    </gazebo>
 </robot>

File: grips_description/urdf/ft_sensor.xacro (robot description, xacro)
@@ -93,5 +93,5 @@
       <plugin name="ft_sensor" filename="libgazebo_ros_ft_sensor.so">
         <robotNamespace>/grips</robotNamespace>
-        <updateRate>100.0</updateRate>
+        <updateRate>1000.0</updateRate>
         <topicName>ft_raw</topicName>
         <jointName>${name}WR</jointName>

File: grips_description/urdf/imu_sensor.xacro (robot description, xacro)
@@ -63,7 +63,8 @@
       <plugin name="imu_sensor" filename="libhector_gazebo_ros_imu.so">
         <robotNamespace>/grips</robotNamespace>
-        <updateRate>500.0</updateRate>
+        <updateRate>1000.0</updateRate>
         <topicName>imu</topicName>
         <bodyName>${prefix}imu_board</bodyName>
+        <gaussianNoise>0.0</gaussianNoise>
       </plugin>
     </gazebo>
